File: AUDIO_OUT.sch (KiCad schematic (older format))
At the start: 25 parts, among them J1 USB_B_Mini, J2 Power, Q1 MMBT2907LT1G, U10 LD1117S33CTR, U2 PCM2900C, Y2 12Mhz

Commit message: delete microSD
Parts:
- removed J2: Power, Pin_Headers:Pin_Header_Straight_1x03_Pitch2.54mm, symbol Conn_01x03
- removed R18: 22R, UI:R_1206_0603, symbol R_Small
- removed U10: LD1117S33CTR, SOT-223, symbol LD1117S33CTR
- added C1, C10, C12, C8, C9: 100nF, UI:C_1206_0603, symbol C_Small
- added C11: 100µF, Capacitors_Tantalum_SMD:CP_Tantalum_Case-D_EIA-7343-31_Wave, symbol CP_Small
- added C13, C14, C15, C16: 2.2µF, Capacitors_Tantalum_SMD:CP_Tantalum_Case-A_EIA-3216-18_Wave, symbol CP_Small
- added J2: IN, UI:audio_jack_3_5mm_PJ307, symbol Audio-Jack-3_2Switches
- added J3: OUT, UI:audio_jack_3_5mm_PJ307, symbol Audio-Jack-3_2Switches
- added L1, L2: 4.7µH, UI:Choke_CD54, symbol L_Small
- added R7: 150R, UI:R_1206_0603, symbol R_Small
- added R8: 300R, UI:R_1206_0603, symbol R_Small
- added U1: LM317_3PinPackage, TO_SOT_Packages_SMD:SOT-223-3_TabPin2, symbol LM317_3PinPackage
- C3: value 10uF -> 47uF; footprint Capacitors_THT:CP_Radial_D5.0mm_P2.00mm -> Capacitors_Tantalum_SMD:CP_Tantalum_Case-D_EIA-7343-31_Wave
- C4, C46, C5, C6: value 100nF -> 1uF
- C49: footprint Capacitors_THT:CP_Radial_D5.0mm_P2.00mm -> Capacitors_Tantalum_SMD:CP_Tantalum_Case-A_EIA-3216-18_Wave
Connections:
- net labels removed: +5V, LINE_IN_LEFT, LINE_IN_RIGHT, LINE_OUT_LEFT, LINE_OUT_RIGHT
- wire segments 88 -> 113
Other:
- moved on the sheet: C2, C3, C4, C46, C49, C5, C50, C6, C7, D1, J1, L4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
