File: LCSDR.sch (KiCad schematic (older format))
At the start: 8 parts, among them J10 Conn_01x01, J11 Conn_01x01, J12 Conn_01x10, J3 Conn_01x10, J4 Conn_01x10, J7 Conn_01x10, J8 Conn_01x01, J9 Conn_01x01

Commit message: delete microSD
Parts:
- removed J10, J11, J8, J9: Conn_01x01, Mounting_Holes:MountingHole_3.2mm_M3_DIN965_Pad, symbol Conn_01x01
- removed J12, J3, J4, J7: Conn_01x10, Pin_Headers:Pin_Header_Straight_1x10_Pitch2.54mm, symbol Conn_01x10
Connections:
- net labels removed: +12V, +9V, BAND, BPF, CLK, GND, I2C_SCL, I2C_SDA, IF_RX_TX, IO0, IO1, IO2, IO3, IO7, IO8, IO9, LINE_IN_LEFT, LINE_IN_RIGHT, LINE_OUT_LEFT, LINE_OUT_RIGHT, MIXER, PTT, ROTATOR, S1_RX_TX, S2_RX_TX
- wire segments 69 -> 0
